Commit message: add RBDL and single leg inverse dynamic controller

File: quadruped_model/urdf/simpledog.urdf (robot description, URDF)
Before this commit: robot simpledog, 17 links, 16 joints
Links:
- link base_link: geometry 
- link front_left_1_Link: geometry 
- link front_left_2_Link: geometry 
- link front_left_3_Link: geometry 
- link front_right_1_Link: geometry 
- link front_right_2_Link: geometry 
- link front_right_3_Link: geometry 
- link lf_foot_Link: geometry 
- link lh_foot_Link: geometry 
- link rear_left_1_Link: geometry 
- link rear_left_2_Link: geometry 
- link rear_left_3_Link: geometry 
- link rear_right_1_Link: geometry 
- link rear_right_2_Link: geometry 
- link rear_right_3_Link: geometry 
- link rf_foot_Link: geometry 
- link rh_foot_Link: geometry 
Joints:
- joint lh_foot_joint: origin xyz=0.24968 0.00033355 -0.015 rpy=0 0 0 -> xyz=0.24742286767759 0.000379574544590811 -0.015 rpy=0 0 0; parent rear_right_3_Link -> rear_left_3_Link
- joint rh_foot_joint: origin xyz=0.24742286767759 0.000379574544590811 -0.015 rpy=0 0 0 -> xyz=0.24968 0.00033355 -0.015 rpy=0 0 0; parent rear_left_3_Link -> rear_right_3_Link
