Commit message: test all legs ID control with EtherCAT Hardware and single_leg_controller, add a template of state_estimate

File: quadruped_model/urdf/quadruped_model.urdf (robot description, URDF)
Before this commit: robot quadruped_model, 17 links, 16 joints
Joints:
- removed joint rf_foot_Link
- added joint rf_foot_joint: type fixed, parent front_right_3_Link, child rf_foot_Link, origin xyz=0.308 0 0.22053 rpy=0 0 0, axis 0 0 0

File: quadruped_model/urdf/quadruped_model_rf_leg.urdf (robot description, URDF)
Before this commit: robot quadruped_model_rf_leg, 5 links, 4 joints
Joints:
- removed joint rf_foot_Link
- added joint rf_foot_joint: type fixed, parent front_right_3_Link, child rf_foot_Link, origin xyz=0.308 0 0.22053 rpy=0 0 0, axis 0 0 0

Commit message: add quadruped_odom for state estimate

File: quadruped_model/urdf/quadruped_model.urdf (robot description, URDF)
Before this commit: robot quadruped_model, 17 links, 16 joints
Joints:
- joint rf_foot_Link: origin xyz=0.308 0 0.22053 rpy=0 0 0 -> xyz=0.308 0 0.23 rpy=0 0 0
- joint rh_foot_joint: origin xyz=0.308 0 0.22053 rpy=0 0 0 -> xyz=0.308 0 0.23 rpy=0 0 0
